Commit message: 修改urdf

File: Xbot/src/simulation/urdf/Xbot.urdf.xacro (robot description, xacro)
@@ -6,5 +6,5 @@
 -->
 <robot name="xbot" xmlns:xacro="http://ros.org/wiki/xacro">
-  <xacro:include filename="./Xbot_base.urdf" />
+  <xacro:include filename="./Xbot_base_rplidar_asus.urdf" />
   <xbot/>
   <sensor_asus_xtion_pro          parent="camera_platform"/>

File: Xbot/src/simulation/urdf/asus_xtion_pro.urdf.xacro (robot description, xacro)
@@ -1,9 +1,7 @@
 <?xml version="1.0"?>
 <robot name="sensor_asus_xtion_pro" xmlns:xacro="http://ros.org/wiki/xacro">
-  <xacro:include filename="$(find turtlebot_description)/urdf/turtlebot_gazebo.urdf.xacro"/>
-  <xacro:include filename="$(find turtlebot_description)/urdf/turtlebot_properties.urdf.xacro"/>
+  <xacro:include filename="$(find simulation)/urdf/common_properties.urdf.xacro"/>
   <!-- Xacro properties -->
   <xacro:property name="M_SCALE" value="0.001"/>
-  <xacro:property name="asus_xtion_pro_cam_py" value="0.0205"/>
   <xacro:property name="asus_xtion_pro_depth_rel_rgb_py" value="0.0270" />
   <xacro:property name="asus_xtion_pro_cam_rel_rgb_py"   value="-0.0220" />
@@ -11,5 +9,5 @@
   <xacro:macro name="sensor_asus_xtion_pro" params="parent">
     <joint name="camera_rgb_joint" type="fixed">
-      <origin xyz="${cam_px} ${asus_xtion_pro_cam_py} ${cam_pz}"
+      <origin xyz="${cam_px} ${cam_py} ${cam_pz}"
               rpy="${cam_or} ${cam_op} ${cam_oy}"/>
       <parent link="${parent}"/>
@@ -33,5 +31,5 @@
         <origin xyz="-0.015 0.0035 0.004" rpy="0 0 0"/>
         <geometry>
-          <mesh filename="package://turtlebot_description/meshes/sensors/xtion_pro_camera.dae"/>
+          <mesh filename="package://simulation/meshes/sensors/xtion_pro_camera.dae"/>
         </geometry>
       </visual>
@@ -66,5 +64,5 @@
     <!-- Asus mount -->
     <joint name="mount_asus_xtion_pro_joint" type="fixed">
-      <origin xyz="-0.1024 0.0 0.272" rpy="0 0 0"/>
+      <origin xyz="-0.02 -0.02 0" rpy="0 0 0"/>
       <parent link="${parent}"/>
       <child link="mount_asus_xtion_pro_link"/>
@@ -74,5 +72,5 @@
         <origin xyz="0 0 0" rpy="${-M_PI/2} 0 0"/>
         <geometry>
-          <mesh filename="package://turtlebot_description/meshes/sensors/xtion_pro_stack.dae"/>
+          <mesh filename="package://simulation/meshes/sensors/xtion_pro_stack.dae"/>
         </geometry>
       </visual>

File: Xbot/src/simulation/urdf/common_properties.urdf.xacro (robot description, xacro)
@@ -4,4 +4,11 @@
  -->
 <robot name="xacro_properties" xmlns:xacro="http://ros.org/wiki/xacro">
+  <property name="cam_px" value="0.0" />
+  <property name="cam_py" value="0.0" />
+  <property name="cam_pz" value="0.025" />
+  <property name="cam_or" value="0" />
+  <property name="cam_op" value="0" />
+  <property name="cam_oy" value="0" />
+  <property name="parent" value="camera_platform" />
   <xacro:property name="M_PI" value="3.1415926535897931" />
   <xacro:property name="material_white">
