Commit message: 123

File: Xbot/src/machine/urdf/turtlebot_properties.urdf.xacro (robot description, xacro)
@@ -22,5 +22,5 @@
 <!--	<xacro:property name="cam_py" value="-0.0125" /> Y varies for different configurations. get sets in sensors_urdf -->
 	<!--<xacro:property name="cam_pz" value="0.43" />-->
-        <xacro:property name="cam_px" value="0.13" />
+        <xacro:property name="cam_px" value="0.12" />
 	<xacro:property name="cam_pz" value="0.87" />
 	<xacro:property name="cam_or" value="0" />
