Commit message: 18.21

File: Xbot/src/machine/urdf/sensors/rplidar.urdf.xacro (robot description, xacro)
@@ -22,5 +22,5 @@
     </link>
     <joint name="base_laser_link" type="fixed">
-      <origin xyz="0.12 0.0 0.15" rpy="0.0 0.0 0.0" />
+      <origin xyz="0.07 0.0 0.21" rpy="0.0 0.0 0.0" />
       <parent link="${parent}" />
       <child link="laser" />
@@ -30,7 +30,7 @@
     <joint name="base_link_to_global_scan" type="fixed">
       <!--<origin xyz="0.0 0.0 0.2" rpy="0 0.0 0.0" />-->
-      <origin xyz="0.12 0.0 0.35" rpy="0 0.0 0.0" />
+      <origin xyz="0.12 0.0 0.56" rpy="0 0.0 0.0" />
       <!--<parent link="base_link" />-->
-      <parent link="laser" />
+      <parent link="${parent}" />
       <child link="global_scan" />
     </joint>
